Commit message: 85

File: src/slam_nav/urdf/ugv_rover.urdf (robot description, URDF)
Before this commit: robot ugv_rover, 13 links, 12 joints
Links:
- link 3d_camera_link: geometry collision mesh filename=file:////home/ws/Desktops/ss/install/slam_nav/share/slam_na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; visual mesh filename=file:////home/ws/Desktops/ss/install/slam_nav/share/slam_na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
- link base_lidar_link: geometry collision mesh filename=file:////home/ws/Desktops/ss/install/slam_nav/share/slam_na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; visual mesh filename=file:////home/ws/Desktops/ss/install/slam_nav/share/slam_na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
- link base_link: geometry collision mesh filename=file:////home/ws/Desktops/ss/install/slam_nav/share/slam_na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; visual mesh filename=file:////home/ws/Desktops/ss/install/slam_nav/share/slam_na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
- link left_down_wheel_link: geometry collision mesh filename=file:////home/ws/Desktops/ss/install/slam_nav/share/slam_na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; visual mesh filename=file:////home/ws/Desktops/ss/install/slam_nav/share/slam_na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
- link left_up_wheel_link: geometry collision mesh filename=file:////home/ws/Desktops/ss/install/slam_nav/share/slam_na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; visual mesh filename=file:////home/ws/Desktops/ss/install/slam_nav/share/slam_na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
- link pt_base_link: geometry collision mesh filename=file:////home/ws/Desktops/ss/install/slam_nav/share/slam_na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; visual mesh filename=file:////home/ws/Desktops/ss/install/slam_nav/share/slam_na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
- link pt_camera_link: geometry collision mesh filename=file:////home/ws/Desktops/ss/install/slam_nav/share/slam_na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; visual mesh filename=file:////home/ws/Desktops/ss/install/slam_nav/share/slam_na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
- link pt_link1: geometry collision mesh filename=file:////home/ws/Desktops/ss/install/slam_nav/share/slam_na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; visual mesh filename=file:////home/ws/Desktops/ss/install/slam_nav/share/slam_na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
- link pt_link2: geometry collision mesh filename=file:////home/ws/Desktops/ss/install/slam_nav/share/slam_na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; visual mesh filename=file:////home/ws/Desktops/ss/install/slam_nav/share/slam_na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
- link right_down_wheel_link: geometry collision mesh filename=file:////home/ws/Desktops/ss/install/slam_nav/share/slam_na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; visual mesh filename=file:////home/ws/Desktops/ss/install/slam_nav/share/slam_na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
- link right_up_wheel_link: geometry collision mesh filename=file:////home/ws/Desktops/ss/install/slam_nav/share/slam_na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; visual mesh filename=file:////home/ws/Desktops/ss/install/slam_nav/share/slam_na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

Commit message: 暂停ldlidar功能包中的tf发布，在整个模型中将雷达统一为base_laser

File: src/slam_nav/urdf/ugv_rover.urdf (robot description, URDF)
Before this commit: robot ugv_rover, 13 links, 12 joints
Links:
- removed link base_lidar_link
- added link base_laser, mass 0.0418000091653573; collision mesh filename=file:////home/ws/Desktops/ss/install/slam_nav/share/slam_na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; visual mesh filename=file:////home/ws/Desktops/ss/install/slam_nav/share/slam_na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
Joints:
- removed joint base_lidar_link_joint
- added joint base_laser_joint: type fixed, parent base_link, child base_laser, origin xyz=0.0398145505519817 0 0.04 rpy=0 0 1.5708, axis 0 0 0

Commit message: VS登封市政府

File: src/slam_nav/urdf/ugv_rover.urdf (robot description, URDF)
Before this commit: robot ugv_rover, 13 links, 12 joints
Joints:
- joint base_laser_joint: origin xyz=0.0398145505519817 0 0.04 rpy=0 0 1.5708 -> xyz=0.0398145505519817 0 0.04 rpy=0 0 0
